Commit message: <fix> left hand direction

File: assets/urdf/shadow_robot/ur10e_shadow_hand_left.urdf (robot description, URDF)
Before this commit: robot ur10e_robot, 43 links, 42 joints
Joints:
- joint left_hand_to_ur10e_base: origin xyz=0 0 0 rpy=0 0 0 -> xyz=0 0 0 rpy=0 0 3.14

File: assets/urdf/shadow_robot/ur10e_shadow_hand_left.xacro (robot description, xacro)
@@ -34,5 +34,5 @@
   <!-- Define the UR10e base link as the parent of the Shadow Hand -->
   <joint name="left_hand_to_ur10e_base" type="fixed">
-    <origin xyz="0 0 0" rpy="0 0 0"/>
+    <origin xyz="0 0 0" rpy="0 0 3.14"/>
     <parent link="tool0"/>
     <child link="lh_forearm"/>
